Commit message: UR5 OK: mundo PRO + cámaras + bridge + panel + scripts
Actualiza paquetes/launch, SDF worlds, scripts de arranque y herramientas UR5. Excluye BORRAR y artefactos runtime.

File: src/ur5_description/urdf/ur5.urdf.xacro (robot description, xacro)
@@ -1,6 +1,122 @@
-<gazebo>
-  <plugin name="gazebo_ros2_control" filename="libgazebo_ros2_control.so">
-    <robot_namespace>/</robot_namespace>
-    <parameters>$(find ur5_description)/config/ur5_controllers.yaml</parameters>
-  </plugin>
-</gazebo>
+<?xml version="1.0"?>
+<!-- URL: /home/laboratorio/TFM/agarre_ros2_ws/src/ur5_description/urdf/ur5.urdf.xacro -->
+<!-- Summary: UR5 description with mock ros2_control and RG2 gripper joints. -->
+<robot xmlns:xacro="http://wiki.ros.org/xacro" name="$(arg name)">
+  <xacro:arg name="name" default="ur5_rg2"/>
+  <xacro:arg name="ur_type" default="ur5"/>
+  <xacro:arg name="tf_prefix" default=""/>
+  <xacro:arg name="joint_limit_params" default="$(find ur_description)/config/$(arg ur_type)/joint_limits.yaml"/>
+  <xacro:arg name="kinematics_params" default="$(find ur_description)/config/$(arg ur_type)/default_kinematics.yaml"/>
+  <xacro:arg name="physical_params" default="$(find ur_description)/config/$(arg ur_type)/physical_parameters.yaml"/>
+  <xacro:arg name="visual_params" default="$(find ur_description)/config/$(arg ur_type)/visual_parameters.yaml"/>
+  <xacro:arg name="safety_limits" default="false"/>
+  <xacro:arg name="safety_pos_margin" default="0.15"/>
+  <xacro:arg name="safety_k_position" default="20"/>
+  <xacro:arg name="force_abs_paths" default="false"/>
+  <xacro:include filename="$(find ur_description)/urdf/ur_macro.xacro"/>
+  <link name="world"/>
+  <xacro:ur_robot
+    name="$(arg name)"
+    tf_prefix="$(arg tf_prefix)"
+    parent="world"
+    joint_limits_parameters_file="$(arg joint_limit_params)"
+    kinematics_parameters_file="$(arg kinematics_params)"
+    physical_parameters_file="$(arg physical_params)"
+    visual_parameters_file="$(arg visual_params)"
+    safety_limits="$(arg safety_limits)"
+    safety_pos_margin="$(arg safety_pos_margin)"
+    safety_k_position="$(arg safety_k_position)"
+    force_abs_paths="$(arg force_abs_paths)"
+    >
+    <origin xyz="0 0 0" rpy="0 0 0"/>
+  </xacro:ur_robot>
+  <!-- RG2 gripper (simplified kinematic stub for ros2_control) -->
+  <link name="rg2_base_link">
+    <inertial>
+      <mass value="0.5"/>
+      <origin xyz="0 0 0" rpy="0 0 0"/>
+      <inertia ixx="0.001" ixy="0.0" ixz="0.0" iyy="0.001" iyz="0.0" izz="0.001"/>
+    </inertial>
+  </link>
+  <joint name="rg2_mount_joint" type="fixed">
+    <parent link="tool0"/>
+    <child link="rg2_base_link"/>
+    <origin xyz="0 0 0" rpy="0 0 0"/>
+  </joint>
+  <link name="rg2_finger_link1">
+    <inertial>
+      <mass value="0.05"/>
+      <origin xyz="0 0 0" rpy="0 0 0"/>
+      <inertia ixx="1e-4" ixy="0.0" ixz="0.0" iyy="1e-4" iyz="0.0" izz="1e-4"/>
+    </inertial>
+  </link>
+  <link name="rg2_finger_link2">
+    <inertial>
+      <mass value="0.05"/>
+      <origin xyz="0 0 0" rpy="0 0 0"/>
+      <inertia ixx="1e-4" ixy="0.0" ixz="0.0" iyy="1e-4" iyz="0.0" izz="1e-4"/>
+    </inertial>
+  </link>
+  <joint name="rg2_finger_joint1" type="prismatic">
+    <parent link="rg2_base_link"/>
+    <child link="rg2_finger_link1"/>
+    <origin xyz="0 0.02 0" rpy="0 0 0"/>
+    <axis xyz="0 1 0"/>
+    <limit lower="0.0" upper="0.04" effort="20" velocity="0.2"/>
+  </joint>
+  <joint name="rg2_finger_joint2" type="prismatic">
+    <parent link="rg2_base_link"/>
+    <child link="rg2_finger_link2"/>
+    <origin xyz="0 -0.02 0" rpy="0 0 0"/>
+    <axis xyz="0 -1 0"/>
+    <limit lower="0.0" upper="0.04" effort="20" velocity="0.2"/>
+  </joint>
+  <!-- ros2_control (mock) with UR5 + RG2 joints -->
+  <ros2_control name="$(arg name)" type="system">
+    <hardware>
+      <plugin>mock_components/GenericSystem</plugin>
+      <param name="state_following_offset">0.0</param>
+      <param name="calculate_dynamics">true</param>
+    </hardware>
+    <joint name="shoulder_pan_joint">
+      <command_interface name="position"/>
+      <state_interface name="position"/>
+      <state_interface name="velocity"/>
+    </joint>
+    <joint name="shoulder_lift_joint">
+      <command_interface name="position"/>
+      <state_interface name="position"/>
+      <state_interface name="velocity"/>
+    </joint>
+    <joint name="elbow_joint">
+      <command_interface name="position"/>
+      <state_interface name="position"/>
+      <state_interface name="velocity"/>
+    </joint>
+    <joint name="wrist_1_joint">
+      <command_interface name="position"/>
+      <state_interface name="position"/>
+      <state_interface name="velocity"/>
+    </joint>
+    <joint name="wrist_2_joint">
+      <command_interface name="position"/>
+      <state_interface name="position"/>
+      <state_interface name="velocity"/>
+    </joint>
+    <joint name="wrist_3_joint">
+      <command_interface name="position"/>
+      <state_interface name="position"/>
+      <state_interface name="velocity"/>
+    </joint>
+    <joint name="rg2_finger_joint1">
+      <command_interface name="position"/>
+      <state_interface name="position"/>
+      <state_interface name="velocity"/>
+    </joint>
+    <joint name="rg2_finger_joint2">
+      <command_interface name="position"/>
+      <state_interface name="position"/>
+      <state_interface name="velocity"/>
+    </joint>
+  </ros2_control>
+</robot>

Commit message: test

File: src/ur5_description/urdf/ur5.urdf.xacro (robot description, xacro)
@@ -2,30 +2,31 @@
 <!-- URL: /home/laboratorio/TFM/agarre_ros2_ws/src/ur5_description/urdf/ur5.urdf.xacro -->
 <!-- Summary: UR5 description with mock ros2_control and RG2 gripper joints. -->
-<robot xmlns:xacro="http://wiki.ros.org/xacro" name="$(arg name)">
-  <xacro:arg name="name" default="ur5_rg2"/>
-  <xacro:arg name="ur_type" default="ur5"/>
-  <xacro:arg name="tf_prefix" default=""/>
-  <xacro:arg name="joint_limit_params" default="$(find ur_description)/config/$(arg ur_type)/joint_limits.yaml"/>
-  <xacro:arg name="kinematics_params" default="$(find ur_description)/config/$(arg ur_type)/default_kinematics.yaml"/>
-  <xacro:arg name="physical_params" default="$(find ur_description)/config/$(arg ur_type)/physical_parameters.yaml"/>
-  <xacro:arg name="visual_params" default="$(find ur_description)/config/$(arg ur_type)/visual_parameters.yaml"/>
-  <xacro:arg name="safety_limits" default="false"/>
-  <xacro:arg name="safety_pos_margin" default="0.15"/>
-  <xacro:arg name="safety_k_position" default="20"/>
-  <xacro:arg name="force_abs_paths" default="false"/>
-  <xacro:include filename="$(find ur_description)/urdf/ur_macro.xacro"/>
+<robot xmlns:xacro="http://wiki.ros.org/xacro" name="ur5_rg2">
+  <xacro:property name="ur_type" value="ur5"/>
+  <xacro:property name="safety_limits" value="false"/>
+  <xacro:property name="safety_pos_margin" value="0.15"/>
+  <xacro:property name="safety_k_position" value="20"/>
+  <xacro:property name="force_abs_paths" value="false"/>
+  <xacro:property name="ur_pkg_share" value="$(optenv UR_DESCRIPTION_SHARE /opt/ros/jazzy/share/ur_description)"/>
+  <xacro:property name="robot_name" value="ur5_rg2"/>
+  <xacro:property name="tf_prefix_value" value=""/>
+  <xacro:property name="joint_limits_file" value="${ur_pkg_share}/config/${ur_type}/joint_limits.yaml"/>
+  <xacro:property name="kinematics_file" value="${ur_pkg_share}/config/${ur_type}/default_kinematics.yaml"/>
+  <xacro:property name="physical_file" value="${ur_pkg_share}/config/${ur_type}/physical_parameters.yaml"/>
+  <xacro:property name="visual_file" value="${ur_pkg_share}/config/${ur_type}/visual_parameters.yaml"/>
+  <xacro:include filename="${ur_pkg_share}/urdf/ur_macro.xacro"/>
   <link name="world"/>
   <xacro:ur_robot
-    name="$(arg name)"
-    tf_prefix="$(arg tf_prefix)"
+    name="${robot_name}"
+    tf_prefix="${tf_prefix_value}"
     parent="world"
-    joint_limits_parameters_file="$(arg joint_limit_params)"
-    kinematics_parameters_file="$(arg kinematics_params)"
-    physical_parameters_file="$(arg physical_params)"
-    visual_parameters_file="$(arg visual_params)"
-    safety_limits="$(arg safety_limits)"
-    safety_pos_margin="$(arg safety_pos_margin)"
-    safety_k_position="$(arg safety_k_position)"
-    force_abs_paths="$(arg force_abs_paths)"
+    joint_limits_parameters_file="${joint_limits_file}"
+    kinematics_parameters_file="${kinematics_file}"
+    physical_parameters_file="${physical_file}"
+    visual_parameters_file="${visual_file}"
+    safety_limits="${safety_limits}"
+    safety_pos_margin="${safety_pos_margin}"
+    safety_k_position="${safety_k_position}"
+    force_abs_paths="${force_abs_paths}"
     >
     <origin xyz="0 0 0" rpy="0 0 0"/>
@@ -73,5 +74,5 @@
   </joint>
   <!-- ros2_control (mock) with UR5 + RG2 joints -->
-  <ros2_control name="$(arg name)" type="system">
+  <ros2_control name="${robot_name}" type="system">
     <hardware>
       <plugin>mock_components/GenericSystem</plugin>
